Commit message: 2402280953

File: source/ext_template/ext_template/assets/MI/mi4/urdf/mi4.urdf (robot description, URDF)
Before this commit: robot mi4, 23 links, 22 joints
Links:
- link FL_thigh_shoulder: geometry 
- link FR_thigh_shoulder: geometry 
- link RL_thigh_shoulder: geometry 
- link RR_thigh_shoulder: geometry 
