Commit message: 2502282337

File: sim2sim_mujoco/robot-descriptions/mi4/urdf/mi4.urdf (robot description, URDF)
Before this commit: robot mi4, 23 links, 22 joints
Links:
- removed link FL_thigh_shoulder
- removed link FR_thigh_shoulder
- removed link RL_thigh_shoulder
- removed link RR_thigh_shoulder
- link FL_calf: geometry collision mesh filename=../meshes/FL_calf.STL scale=1 1 1; visual mesh filename=../meshes/FL_calf.STL scale=1 1 1
- link FL_hip: geometry collision cylinder length=0.065 radius=0.065; visual mesh filename=../meshes/FL_hip.STL scale=1 1 1
- link FL_thigh: geometry collision box size=0.35 0.04 0.04; visual mesh filename=../meshes/FL_thigh.STL scale=1 1 1
- link FR_calf: geometry collision mesh filename=../meshes/FR_calf.STL scale=1 1 1; visual mesh filename=../meshes/FR_calf.STL scale=1 1 1
- link FR_hip: geometry collision mesh filename=../meshes/FR_hip.STL scale=1 1 1; visual mesh filename=../meshes/FR_hip.STL scale=1 1 1
- link FR_thigh: geometry collision mesh filename=../meshes/FR_thigh.STL scale=1 1 1; visual mesh filename=../meshes/FR_thigh.STL scale=1 1 1
- link RL_calf: geometry collision mesh filename=../meshes/RL_calf.STL scale=1 1 1; visual mesh filename=../meshes/RL_calf.STL scale=1 1 1
- link RL_hip: geometry collision mesh filename=../meshes/RL_hip.STL scale=1 1 1; visual mesh filename=../meshes/RL_hip.STL scale=1 1 1
- link RL_thigh: geometry collision mesh filename=../meshes/RL_thigh.STL scale=1 1 1; visual mesh filename=../meshes/RL_thigh.STL scale=1 1 1
- link RR_calf: geometry collision mesh filename=../meshes/RR_calf.STL scale=1 1 1; visual mesh filename=../meshes/RR_calf.STL scale=1 1 1
- link RR_hip: geometry collision mesh filename=../meshes/RR_hip.STL scale=1 1 1; visual mesh filename=../meshes/RR_hip.STL scale=1 1 1
- link RR_thigh: geometry collision mesh filename=../meshes/RR_thigh.STL scale=1 1 1; visual mesh filename=../meshes/RR_thigh.STL scale=1 1 1
- link base: mass None -> 0.001
- link imu_link: geometry collision box size=.001 .001 .001; visual box size=0.001 0.001 0.001
Joints:
- removed joint FL_hip_fixed
- removed joint FR_hip_fixed
- removed joint RL_hip_fixed
- removed joint RR_hip_fixed
